File: ESCv4.3.kicad_pcb (KiCad board)
At the start: 4 copper layers, 40 x 38.1 mm, 109 parts, among them J1 PWR_IN, J3 Conn_01x10, J4 SPI1, J5 Conn_01x05, J6 CAN1, J7 CAN2, J7_1 Phase_Pads, J8 Conn_01x05, Q2 BC847BTT1G, Q4 CSD25501F3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

Commit message: first commit
Other:
- net class CAN removed
- net class Default removed
- net class TEMPSENSE removed
- net class VDD removed

Commit message: production version v1
Parts:
- removed C21, C22: 22uF 16V, Capacitor_SMD:C_0603_1608Metric
- added R8: 2k2, Resistor_SMD:R_0402_1005Metric, F.Cu at (93.1, 97.6)
- C14: value 10uF 50V -> 4.7uF 50V
- C15: value 10uF 50V -> 100nF 50V 5%; footprint Capacitor_SMD:C_0805_2012Metric -> Capacitor_SMD:C_0402_1005Metric
- C16: value 100nF 50V 5% -> 1uF 50V
- J8: value Conn_01x05 -> Conn_01x04
- L1: value 1µH -> 4.7uH; footprint Inductor_SMD:L_Coilcraft_XxL4020 -> Inductor_SMD:L_Coilcraft_XxL4030
- R11: value 1MΩ -> 200k 1%; moved to F.Cu
- R15: value 2k2 -> 47k 1%
- SW1, SW2: footprint runger:USLPT2616CT2TR -> runger:NANOT240
- U1: value TPS63061 -> MAX20076; footprint Package_SON:Texas_S-PWSON-N10_ThermalVias -> runger:DFN-12-1EP_3x3mm_P0.5mm_EP1.7x2.5mm
- U3: value MCP2542WFDxMF -> TJA1051TK/3
- U7: value MA732 -> AS5047P; footprint Package_DFN_QFN:QFN-16-1EP_3x3mm_P0.5mm_EP1.75x1.75mm -> Package_SO:TSSOP-14_4.4x5mm_P0.65mm
- moved C14 6.90 mm to (83.2, 95.0)
- moved C16 6.83 mm to (90.5, 94.7), turned to 180 degrees
- moved L1 6.35 mm to (86.4, 99.5), turned to 0 degrees
- moved C15 5.95 mm to (84.2, 96.5)
- moved C20 5.68 mm to (92.1, 95.9), turned to 0 degrees
- moved R11 5.07 mm to (90.0, 96.2)
- moved D4 3.00 mm to (92.1, 97.6), turned to 90 degrees
- moved R15 2.47 mm to (89.6, 97.7), turned to 180 degrees
- moved C39 2.13 mm to (104.4, 100.8)
- moved R23 1.02 mm to (97.6, 93.7)
- moved U1 0.48 mm to (87.3, 95.3), turned to 0 degrees
- moved R28 0.22 mm to (107.3, 98.5)
- moved C35 0.22 mm to (107.3, 99.5)
- moved G*** 0.21 mm to (89.7, 104.3)
- moved FB1 0.10 mm to (90.1, 90.8)
Connections:
- C15 pad 1: Net-(C14-Pad1) -> Net-(C15-Pad1)
- C15 pad 2: GND -> Net-(C15-Pad2)
- C16 pad 1: Net-(C16-Pad1) -> GND
- C16 pad 2: GND -> Net-(C16-Pad2)
- J3 pad 10: Net-(J3-Pad10) -> unconnected-(J3-Pad10) (x2)
- J3 pad 3: Net-(J3-Pad3) -> unconnected-(J3-Pad3) (x2)
- J3 pad 4: Net-(J3-Pad4) -> unconnected-(J3-Pad4) (x2)
- J3 pad 9: Net-(J3-Pad9) -> unconnected-(J3-Pad9) (x2)
- L1 pad 1: Net-(L1-Pad1) -> Net-(C15-Pad1)
- L1 pad 2: Net-(L1-Pad2) -> +5VD
- R11 pad 1: Net-(R11-Pad1) -> +5VD
- R11 pad 2: +5VD -> Net-(R11-Pad2)
- R15 pad 1: GND -> Net-(R11-Pad2)
- R15 pad 2: Net-(D4-Pad1) -> GND
- U1 pad 1: Net-(L1-Pad1) -> unconnected-(U1-Pad1)
- U1 pad 10: Net-(L1-Pad2) -> Net-(C16-Pad2)
- U1 pad 11: GND -> unconnected-(U1-Pad11)
- U1 pad 3: Net-(C14-Pad1) -> Net-(C15-Pad2)
- U1 pad 4: GND -> Net-(C14-Pad1)
- U1 pad 5: Net-(R11-Pad1) -> Net-(C15-Pad1)
- U1 pad 6: Net-(C16-Pad1) -> GND
- U1 pad 8: +5VD -> Net-(R11-Pad2)
- U5 pad 1: Net-(U5-Pad1) -> unconnected-(U5-Pad1)
- U5 pad 24: Net-(U5-Pad24) -> unconnected-(U5-Pad24)
- U6 pad 2: Net-(U6-Pad2) -> unconnected-(U6-Pad2)
- U6 pad 25: Net-(U6-Pad25) -> unconnected-(U6-Pad25)
- U6 pad 26: Net-(U6-Pad26) -> unconnected-(U6-Pad26)
- U6 pad 27: Net-(U6-Pad27) -> unconnected-(U6-Pad27)
- U6 pad 30: Net-(U6-Pad30) -> unconnected-(U6-Pad30)
- U6 pad 31: Net-(U6-Pad31) -> unconnected-(U6-Pad31)
- U6 pad 32: Net-(U6-Pad32) -> unconnected-(U6-Pad32)
- U6 pad 33: Net-(U6-Pad33) -> unconnected-(U6-Pad33)
- U6 pad 44: Net-(U6-Pad44) -> unconnected-(U6-Pad44)
- U6 pad 45: Net-(U6-Pad45) -> unconnected-(U6-Pad45)
- U6 pad 47: Net-(U6-Pad47) -> unconnected-(U6-Pad47)
- U6 pad 48: Net-(U6-Pad48) -> unconnected-(U6-Pad48)
- U7 pad 1: Net-(U7-Pad1) -> /nCS2
- U7 pad 10: GND -> unconnected-(U7-Pad10)
- U7 pad 11: Net-(U7-Pad11) -> VDD
- U7 pad 12: /SCLK -> VDD
- U7 pad 13: VDD -> GND
- U7 pad 14: Net-(U7-Pad14) -> /ABI_I
- U7 pad 2: /ABI_A -> /SCLK
- U7 pad 3: /ABI_I -> /MISO
- U7 pad 5: /nCS2 -> GND
- U7 pad 7: /MISO -> /ABI_A
- U7 pad 8: GND -> unconnected-(U7-Pad8)
- U7 pad 9: Net-(U7-Pad9) -> unconnected-(U7-Pad9)
Routing:
- net GND: track 168.6 -> 152.0 mm, vias 22 -> 26
- net /nCS2: track 4.19 -> 12.2 mm
- net /ABI_I: track 16.0 -> 8.23 mm
- net Net-(C14-Pad1): track 6.67 -> 12.5 mm
- net Net-(C15-Pad1): track 0.00 -> 4.47 mm
- net /SDA1: track 39.5 -> 43.9 mm
- net /MISO: track 25.0 -> 29.2 mm
- net Net-(C15-Pad2): track 0.00 -> 3.95 mm, vias 0 -> 2
- net /ABI_A: track 16.7 -> 12.9 mm
- net Net-(L1-Pad2): track 3.23 -> 0.00 mm
- net Net-(L1-Pad1): track 3.22 -> 0.00 mm
- net /ABI_B: track 6.98 -> 9.89 mm
- net +5VD: track 36.8 -> 34.0 mm
- net Net-(J3-Pad3): track 2.58 -> 0.00 mm, vias 1 -> 0
- net unconnected-(J3-Pad4): track 0.00 -> 2.57 mm, vias 0 -> 1
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- added copper zone on F.Cu, net GND
Other:
- rule pad_to_mask_clearance: 0.05 -> 0
- board text added: "H"
- board text added: "L"
- board text added: "max 35V 3A"
- board text added: "v2.0 ©2022 runger"
- board text removed: "max 40V 3A"
- board text removed: "v2.0 ©2021 runger"
