File: ESCv4.3.kicad_sch (KiCad schematic)
At the start: 84 parts, among them J1 PWR_IN, J3 Conn_01x10, J4 SPI1, J5 Conn_01x05, J6 CAN1, J7 CAN2, J7_1 Phase_Pads, J8 Conn_01x05, Q2 BC847BTT1G, Q4 CSD25501F3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

Commit message: production version v1
Parts:
- removed C14, C15: 10uF 50V, Capacitor_SMD:C_0805_2012Metric, symbol Device:C_Small
- removed C16: 100nF 50V 5%, Capacitor_SMD:C_0402_1005Metric, symbol Device:C_Small
- removed C20, C21, C22: 22uF 16V, Capacitor_SMD:C_0603_1608Metric, symbol Device:C_Small
- removed FB1: 180Ω@100Mhz, Inductor_SMD:L_0805_2012Metric, symbol Device:Ferrite_Bead
- removed L1: 1uH, Inductor_SMD:L_Coilcraft_XxL4020, symbol Device:L
- removed R11: 1MΩ, Resistor_SMD:R_0402_1005Metric, symbol Device:R_Small
- removed R15: 2k2, Resistor_SMD:R_0402_1005Metric, symbol Device:R_Small
- removed U1: TPS63061, Package_SON:Texas_S-PWSON-N10_ThermalVias, symbol runger:TPS63061
- removed U7: MA732, Package_DFN_QFN:QFN-16-1EP_3x3mm_P0.5mm_EP1.75x1.75mm, symbol Sensor_Magnetic:MA730
- added R8: 2k2, Resistor_SMD:R_0402_1005Metric, symbol Device:R_Small
- added U7: AS5047P, Package_SO:TSSOP-14_4.4x5mm_P0.65mm, symbol Sensor_Magnetic:AS5047D
- J8: value Conn_01x05 -> Conn_01x04
- SW1: footprint runger:USLPT2616CT2TR -> runger:NANOT240
- SW2: footprint runger:USLPT2616CT2TR -> runger:NANOT240; Manu TE Connectivity / Alcoswitch -> C&K Switches; Part USLPT2616CT2TR -> NANOT240
- U3: value MCP2542WFDxMF -> TJA1051TK/3; Manu Microchip -> NXP; Part MCP2542WFDxMF -> TJA1051TK/3
Connections:
- net ABI_A: now also U7.7 (A)
- net ABI_B: now also U7.6 (B)
- net ABI_I: now also U7.14 (I/PWM)
- net GND: now also SW2.1, R8.1, U7.13 (GND), U7.5 (TST); no longer R12.2
- net MISO: now also U7.3 (MISO)
- net MOSI: now also U7.4 (MOSI)
- net SCLK: now also U7.2 (CLK)
- net VDD: now also R12.2, U7.11 (VDD), U7.12 (VDD3V3); no longer SW2.1
- net nCS2: now also U7.1 (~{CS})
- net at D4.1 (K): now also R8.2
- no-connect marks 17 -> 16
Other:
- added sheet Buck_MAX20076 (Buck_MAX20076.kicad_sch)
- note removed: "Add IO1 port"
- note removed: "Add filters, add RX/TX LEDs"
- note removed: "Check FET thresholds"
- note removed: "Pick LEDs and check currents"
- moved on the sheet: C19, C39, R12, SW2
